File: hardware/pcb/analyzer/Trimix_Analyzer.kicad_pcb (KiCad board)
At the start: 4 copper layers, 30 x 99 mm, 169 parts, among them J101 USB HARNESS: 5V/GND/CC1/CC2/D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, J102 PACK PIGTAIL, J103 PACK NTC: 103AT-2, J104 ARM: OPEN, J301 GUITION JP1 / 2x13, J401 AO2 / 3-pin cable, J402 SMB male-centre / Amphenol142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, J501 MD62 cable / <=30 cm, J601 BME280 harness, J701 ZE07-CO harness, J801 POWER BUTTON / 1NO, J802 BUTTON LED +/-, Q101 2N7002, Q110 DMN2056U-7, Q111 DMN2056U-7, Q112 DMN2056U-7, Q601 BSS138, Q602 BSS138, U101 BQ25895RTWR, U110 TUSB320LAIRWBR, U111 PI3USB9201ZTAEX, U112 SN74AUP1G74DCUR, U113 TPS3808G01DBVR, U114 TPS22950CQDDCRQ1, U115 TPS259470ARPWR, U201 TPS63020DSJR, U301 MAX17048G+, U302 LM66100DCKR, U401 ADS122C04IPWR, U501 TPS7A2030PDBVR, U502 ADS122C04IPWR, U701 TPS61023DRLR, U702 TPS7A2030PDBVR, U703 TXU0202DCUR, U801 LTC2954CTS8-1

Commit message: Add files via upload
Changes on all for layers of the PCB
Optimized the placing of some components for shorter routing
Rotaded the 3-pin HE-connector (J501) for 180°
Parts:
- C103: moved to F.Cu
- C111, C112, C113, R112: moved to B.Cu
- moved C402 36.4 mm to (28.1, 51.2), turned to -90 degrees
- moved C401 36.4 mm to (28.1, 47.9)
- moved C501 33.9 mm to (23.9, 70.2)
- moved J501 33.2 mm to (23.9, 61.5), turned to 180 degrees
- moved R115 31.2 mm to (42.4, 106.4), turned to 90 degrees
- moved C706 31.0 mm to (23.9, 86.5)
- moved C103 31.0 mm to (36.0, 103.1), turned to 0 degrees
- moved C702 30.7 mm to (40.8, 78.0), turned to 180 degrees
- moved R702 30.7 mm to (38.4, 77.9), turned to -90 degrees
- moved C113 30.2 mm to (48.5, 103.5)
- moved R406 30.1 mm to (31.2, 39.9), turned to 0 degrees
- moved C112 29.6 mm to (48.6, 107.3), turned to -90 degrees
- moved R119 29.5 mm to (25.1, 109.9)
- moved C407 29.4 mm to (31.1, 50.0)
- moved R407 29.4 mm to (31.1, 51.7)
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Routing:
- net HOST_3V3: track 239.9 -> 59.7 mm, vias 15 -> 31
- net VOUT_5V: track 118.2 -> 12.7 mm, vias 10 -> 14
- net VSYS: track 141.9 -> 80.1 mm, vias 12 -> 6
- net USB_5V: track 125.2 -> 79.1 mm, vias 9 -> 3
- net USB_D_P: track 72.5 -> 36.0 mm, vias 6 -> 0
- net O2_B_RAW_N: track 35.2 -> 3.61 mm, vias 1 -> 11
- net HE_3V0: track 47.4 -> 16.1 mm, vias 2 -> 0
- net CHG_INT_N: track 110.9 -> 81.3 mm, vias 8 -> 4
- net GND: track 176.2 -> 150.8 mm, vias 72 -> 92
- net USB_ILIM_AUTH: track 64.5 -> 40.8 mm, vias 4 -> 2
- net I2C_SDA: track 140.4 -> 120.3 mm, vias 8 -> 7
- net O2_B_RAW_P: track 23.7 -> 6.79 mm
- net /01  CHARGING + BATTERY/BQ_REGN: track 38.6 -> 24.1 mm, vias 4 -> 2
- net BME_SCL: track 76.5 -> 64.7 mm, vias 3 -> 6
- net USB_ILIM_BRANCH: track 25.6 -> 14.0 mm, vias 3 -> 2
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- added copper zone on F.Cu, net /01  CHARGING + BATTERY/BQ_SW
- added copper zone on In2.Cu, net HOST_3V3
- added copper zone on B.Cu, net O2_B_RAW_N
- added copper zone on In1.Cu, net O2_B_RAW_N
- added copper zone on B.Cu, net VOUT_5V
- added copper zone on F.Cu, net VOUT_5V
- added copper zone on F.Cu, net VSYS
- removed copper zone on In2.Cu, net GND
